Commit message: changed the paths of meshes in robot urdf files

File: models/data/robots/franka_panda/panda.urdf (robot description, URDF)
Before this commit: robot panda, 12 links, 11 joints
Links:
- link panda_hand: geometry collision mesh filename=package://robots/franka_panda/meshes/collision/hand.stl; visual mesh filename=package://robots/franka_panda/meshes/visual/hand.dae
- link panda_leftfinger: geometry collision mesh filename=package://robots/franka_panda/meshes/collision/finger.stl; visual mesh filename=package://robots/franka_panda/meshes/visual/finger.dae
- link panda_link0: geometry collision mesh filename=package://robots/franka_panda/meshes/collision/link0.stl; visual mesh filename=package://robots/franka_panda/meshes/visual/link0.dae
- link panda_link1: geometry collision mesh filename=package://robots/franka_panda/meshes/collision/link1.stl; visual mesh filename=package://robots/franka_panda/meshes/visual/link1.dae
- link panda_link2: geometry collision mesh filename=package://robots/franka_panda/meshes/collision/link2.stl; visual mesh filename=package://robots/franka_panda/meshes/visual/link2.dae
- link panda_link3: geometry collision mesh filename=package://robots/franka_panda/meshes/collision/link3.stl; visual mesh filename=package://robots/franka_panda/meshes/visual/link3.dae
- link panda_link4: geometry collision mesh filename=package://robots/franka_panda/meshes/collision/link4.stl; visual mesh filename=package://robots/franka_panda/meshes/visual/link4.dae
- link panda_link5: geometry collision mesh filename=package://robots/franka_panda/meshes/collision/link5.stl; visual mesh filename=package://robots/franka_panda/meshes/visual/link5.dae
- link panda_link6: geometry collision mesh filename=package://robots/franka_panda/meshes/collision/link6.stl; visual mesh filename=package://robots/franka_panda/meshes/visual/link6.dae
- link panda_link7: geometry collision mesh filename=package://robots/franka_panda/meshes/collision/link7.stl; visual mesh filename=package://robots/franka_panda/meshes/visual/link7.dae
- link panda_rightfinger: geometry collision mesh filename=package://robots/franka_panda/meshes/collision/finger.stl; visual mesh filename=package://robots/franka_panda/meshes/visual/finger.dae

File: models/data/robots/kuka_iiwa/kuka_iiwa.urdf (robot description, URDF)
Before this commit: robot iiwa, 12 links, 11 joints
Links:
- link iiwa_link_0: geometry collision mesh filename=package://robots/kuka_iiwa/meshes/collision/link_0.stl; visual mesh filename=package://robots/kuka_iiwa/meshes/visual/link_0.stl
- link iiwa_link_1: geometry collision mesh filename=package://robots/kuka_iiwa/meshes/collision/link_1.stl; visual mesh filename=package://robots/kuka_iiwa/meshes/visual/link_1.stl
- link iiwa_link_2: geometry collision mesh filename=package://robots/kuka_iiwa/meshes/collision/link_2.stl; visual mesh filename=package://robots/kuka_iiwa/meshes/visual/link_2.stl
- link iiwa_link_3: geometry collision mesh filename=package://robots/kuka_iiwa/meshes/collision/link_3.stl; visual mesh filename=package://robots/kuka_iiwa/meshes/visual/link_3.stl
- link iiwa_link_4: geometry collision mesh filename=package://robots/kuka_iiwa/meshes/collision/link_4.stl; visual mesh filename=package://robots/kuka_iiwa/meshes/visual/link_4.stl
- link iiwa_link_5: geometry collision mesh filename=package://robots/kuka_iiwa/meshes/collision/link_5.stl; visual mesh filename=package://robots/kuka_iiwa/meshes/visual/link_5.stl
- link iiwa_link_6: geometry collision mesh filename=package://robots/kuka_iiwa/meshes/collision/link_6.stl; visual mesh filename=package://robots/kuka_iiwa/meshes/visual/link_6.stl
- link iiwa_link_7: geometry collision mesh filename=package://robots/kuka_iiwa/meshes/collision/link_7_basic.stl; visual mesh filename=package://robots/kuka_iiwa/meshes/visual/link_7_basic.stl
- link panda_hand: geometry collision mesh filename=package://robots/franka_panda/meshes/collision/hand.stl; visual mesh filename=package://robots/franka_panda/meshes/visual/hand.dae
- link panda_leftfinger: geometry collision mesh filename=package://robots/franka_panda/meshes/collision/finger.stl; visual mesh filename=package://robots/franka_panda/meshes/visual/finger.dae
- link panda_rightfinger: geometry collision mesh filename=package://robots/franka_panda/meshes/collision/finger.stl; visual mesh filename=package://robots/franka_panda/meshes/visual/finger.dae

File: models/data/robots/kuka_kmr_iiwa/kuka_kmr_iiwa.urdf (robot description, URDF)
Before this commit: robot kmr_iiwa, 16 links, 15 joints
Links:
- link iiwa_link_0: geometry collision mesh filename=package://robots/kuka_iiwa/meshes/collision/link_0.stl; visual mesh filename=package://robots/kuka_iiwa/meshes/visual/link_0.stl
- link iiwa_link_1: geometry collision mesh filename=package://robots/kuka_iiwa/meshes/collision/link_1.stl; visual mesh filename=package://robots/kuka_iiwa/meshes/visual/link_1.stl
- link iiwa_link_2: geometry collision mesh filename=package://robots/kuka_iiwa/meshes/collision/link_2.stl; visual mesh filename=package://robots/kuka_iiwa/meshes/visual/link_2.stl
- link iiwa_link_3: geometry collision mesh filename=package://robots/kuka_iiwa/meshes/collision/link_3.stl; visual mesh filename=package://robots/kuka_iiwa/meshes/visual/link_3.stl
- link iiwa_link_4: geometry collision mesh filename=package://robots/kuka_iiwa/meshes/collision/link_4.stl; visual mesh filename=package://robots/kuka_iiwa/meshes/visual/link_4.stl
- link iiwa_link_5: geometry collision mesh filename=package://robots/kuka_iiwa/meshes/collision/link_5.stl; visual mesh filename=package://robots/kuka_iiwa/meshes/visual/link_5.stl
- link iiwa_link_6: geometry collision mesh filename=package://robots/kuka_iiwa/meshes/collision/link_6.stl; visual mesh filename=package://robots/kuka_iiwa/meshes/visual/link_6.stl
- link iiwa_link_7: geometry collision mesh filename=package://robots/kuka_iiwa/meshes/collision/link_7_basic.stl; visual mesh filename=package://robots/kuka_iiwa/meshes/visual/link_7_basic.stl
- link kmr_link: geometry collision box size=1.122 0.631 0.701; visual mesh filename=package://robots/kuka_kmr_iiwa/meshes/visual/kmr.stl scale=0.001 0.001 0.001
- link panda_hand: geometry collision mesh filename=package://robots/franka_panda/meshes/collision/hand.stl; visual mesh filename=package://robots/franka_panda/meshes/visual/hand.dae
- link panda_leftfinger: geometry collision mesh filename=package://robots/franka_panda/meshes/collision/finger.stl; visual mesh filename=package://robots/franka_panda/meshes/visual/finger.dae
- link panda_rightfinger: geometry collision mesh filename=package://robots/franka_panda/meshes/collision/finger.stl; visual mesh filename=package://robots/franka_panda/meshes/visual/finger.dae

File: models/data/robots/ur5/ur5.urdf (robot description, URDF)
Before this commit: robot ur5, 11 links, 10 joints
Links:
- link base_link: geometry collision mesh filename=package://robots/ur5/meshes/collision/base.stl; visual mesh filename=package://robots/ur5/meshes/visual/base.dae
- link forearm_link: geometry collision mesh filename=package://robots/ur5/meshes/collision/forearm.stl; visual mesh filename=package://robots/ur5/meshes/visual/forearm.dae
- link panda_hand: geometry collision mesh filename=package://robots/franka_panda/meshes/collision/hand.stl; visual mesh filename=package://robots/franka_panda/meshes/visual/hand.dae
- link panda_leftfinger: geometry collision mesh filename=package://robots/franka_panda/meshes/collision/finger.stl; visual mesh filename=package://robots/franka_panda/meshes/visual/finger.dae
- link panda_rightfinger: geometry collision mesh filename=package://robots/franka_panda/meshes/collision/finger.stl; visual mesh filename=package://robots/franka_panda/meshes/visual/finger.dae
- link shoulder_link: geometry collision mesh filename=package://robots/ur5/meshes/collision/shoulder.stl; visual mesh filename=package://robots/ur5/meshes/visual/shoulder.dae
- link upper_arm_link: geometry collision mesh filename=package://robots/ur5/meshes/collision/upperarm.stl; visual mesh filename=package://robots/ur5/meshes/visual/upperarm.dae
- link wrist_1_link: geometry collision mesh filename=package://robots/ur5/meshes/collision/wrist1.stl; visual mesh filename=package://robots/ur5/meshes/visual/wrist1.dae
- link wrist_2_link: geometry collision mesh filename=package://robots/ur5/meshes/collision/wrist2.stl; visual mesh filename=package://robots/ur5/meshes/visual/wrist2.dae
- link wrist_3_link: geometry collision mesh filename=package://robots/ur5/meshes/collision/wrist3.stl; visual mesh filename=package://robots/ur5/meshes/visual/wrist3.dae
