Commit message: Small changes I was making to make planner run

File: src/guided_tamp_benchmark/models/data/robots/franka_panda/panda.urdf (robot description, URDF)
Before this commit: robot panda, 12 links, 11 joints
Links:
- link panda_hand: geometry collision mesh filename=package://data/robots/franka_panda/meshes/collision/hand.stl; visual mesh filename=package://data/robots/franka_panda/meshes/visual/hand.dae
- link panda_leftfinger: geometry collision mesh filename=package://data/robots/franka_panda/meshes/collision/finger.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; visual mesh filename=package://data/robots/franka_panda/meshes/visual/finger.dae
- link panda_link0: geometry collision mesh filename=package://data/robots/franka_panda/meshes/collision/link0.s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; visual mesh filename=package://data/robots/franka_panda/meshes/visual/link0.dae
- link panda_link1: geometry collision mesh filename=package://data/robots/franka_panda/meshes/collision/link1.s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; visual mesh filename=package://data/robots/franka_panda/meshes/visual/link1.dae
- link panda_link2: geometry collision mesh filename=package://data/robots/franka_panda/meshes/collision/link2.s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; visual mesh filename=package://data/robots/franka_panda/meshes/visual/link2.dae
- link panda_link3: geometry collision mesh filename=package://data/robots/franka_panda/meshes/collision/link3.s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; visual mesh filename=package://data/robots/franka_panda/meshes/visual/link3.dae
- link panda_link4: geometry collision mesh filename=package://data/robots/franka_panda/meshes/collision/link4.s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; visual mesh filename=package://data/robots/franka_panda/meshes/visual/link4.dae
- link panda_link5: geometry collision mesh filename=package://data/robots/franka_panda/meshes/collision/link5.s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; visual mesh filename=package://data/robots/franka_panda/meshes/visual/link5.dae
- link panda_link6: geometry collision mesh filename=package://data/robots/franka_panda/meshes/collision/link6.s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; visual mesh filename=package://data/robots/franka_panda/meshes/visual/link6.dae
- link panda_link7: geometry collision mesh filename=package://data/robots/franka_panda/meshes/collision/link7.s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; visual mesh filename=package://data/robots/franka_panda/meshes/visual/link7.dae
- link panda_rightfinger: geometry collision mesh filename=package://data/robots/franka_panda/meshes/collision/finger.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; visual mesh filename=package://data/robots/franka_panda/meshes/visual/finger.dae

File: src/guided_tamp_benchmark/models/data/robots/ur5/ur5.urdf (robot description, URDF)
Before this commit: robot ur5, 11 links, 10 joints
Links:
- link base_link: geometry collision mesh filename=package://data/robots/ur5/meshes/collision/base.stl; visual mesh filename=package://data/robots/ur5/meshes/visual/base.dae
- link forearm_link: geometry collision mesh filename=package://data/robots/ur5/meshes/collision/forearm.stl; visual mesh filename=package://data/robots/ur5/meshes/visual/forearm.dae
- link panda_hand: geometry collision mesh filename=package://data/robots/franka_panda/meshes/collision/hand.stl; visual mesh filename=package://data/robots/franka_panda/meshes/visual/hand.dae
- link panda_leftfinger: geometry collision mesh filename=package://data/robots/franka_panda/meshes/collision/finger.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; visual mesh filename=package://data/robots/franka_panda/meshes/visual/finger.dae
- link panda_rightfinger: geometry collision mesh filename=package://data/robots/franka_panda/meshes/collision/finger.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; visual mesh filename=package://data/robots/franka_panda/meshes/visual/finger.dae
- link shoulder_link: geometry collision mesh filename=package://data/robots/ur5/meshes/collision/shoulder.stl; visual mesh filename=package://data/robots/ur5/meshes/visual/shoulder.dae
- link upper_arm_link: geometry collision mesh filename=package://data/robots/ur5/meshes/collision/upperarm.stl; visual mesh filename=package://data/robots/ur5/meshes/visual/upperarm.dae
- link wrist_1_link: geometry collision mesh filename=package://data/robots/ur5/meshes/collision/wrist1.stl; visual mesh filename=package://data/robots/ur5/meshes/visual/wrist1.dae
- link wrist_2_link: geometry collision mesh filename=package://data/robots/ur5/meshes/collision/wrist2.stl; visual mesh filename=package://data/robots/ur5/meshes/visual/wrist2.dae
- link wrist_3_link: geometry collision mesh filename=package://data/robots/ur5/meshes/collision/wrist3.stl; visual mesh filename=package://data/robots/ur5/meshes/visual/wrist3.dae

Commit message: Revert stupid change

File: src/guided_tamp_benchmark/models/data/robots/franka_panda/panda.urdf (robot description, URDF)
Before this commit: robot panda, 12 links, 11 joints
Links:
- link panda_hand: geometry collision mesh filename=package://robots/franka_panda/meshes/collision/hand.stl; visual mesh filename=package://robots/franka_panda/meshes/visual/hand.dae
- link panda_leftfinger: geometry collision mesh filename=package://robots/franka_panda/meshes/collision/finger.stl; visual mesh filename=package://robots/franka_panda/meshes/visual/finger.dae
- link panda_link0: geometry collision mesh filename=package://robots/franka_panda/meshes/collision/link0.stl; visual mesh filename=package://robots/franka_panda/meshes/visual/link0.dae
- link panda_link1: geometry collision mesh filename=package://robots/franka_panda/meshes/collision/link1.stl; visual mesh filename=package://robots/franka_panda/meshes/visual/link1.dae
- link panda_link2: geometry collision mesh filename=package://robots/franka_panda/meshes/collision/link2.stl; visual mesh filename=package://robots/franka_panda/meshes/visual/link2.dae
- link panda_link3: geometry collision mesh filename=package://robots/franka_panda/meshes/collision/link3.stl; visual mesh filename=package://robots/franka_panda/meshes/visual/link3.dae
- link panda_link4: geometry collision mesh filename=package://robots/franka_panda/meshes/collision/link4.stl; visual mesh filename=package://robots/franka_panda/meshes/visual/link4.dae
- link panda_link5: geometry collision mesh filename=package://robots/franka_panda/meshes/collision/link5.stl; visual mesh filename=package://robots/franka_panda/meshes/visual/link5.dae
- link panda_link6: geometry collision mesh filename=package://robots/franka_panda/meshes/collision/link6.stl; visual mesh filename=package://robots/franka_panda/meshes/visual/link6.dae
- link panda_link7: geometry collision mesh filename=package://robots/franka_panda/meshes/collision/link7.stl; visual mesh filename=package://robots/franka_panda/meshes/visual/link7.dae
- link panda_rightfinger: geometry collision mesh filename=package://robots/franka_panda/meshes/collision/finger.stl; visual mesh filename=package://robots/franka_panda/meshes/visual/finger.dae

File: src/guided_tamp_benchmark/models/data/robots/ur5/ur5.urdf (robot description, URDF)
Before this commit: robot ur5, 11 links, 10 joints
Links:
- link base_link: geometry collision mesh filename=package://robots/ur5/meshes/collision/base.stl; visual mesh filename=package://robots/ur5/meshes/visual/base.dae
- link forearm_link: geometry collision mesh filename=package://robots/ur5/meshes/collision/forearm.stl; visual mesh filename=package://robots/ur5/meshes/visual/forearm.dae
- link panda_hand: geometry collision mesh filename=package://robots/franka_panda/meshes/collision/hand.stl; visual mesh filename=package://robots/franka_panda/meshes/visual/hand.dae
- link panda_leftfinger: geometry collision mesh filename=package://robots/franka_panda/meshes/collision/finger.stl; visual mesh filename=package://robots/franka_panda/meshes/visual/finger.dae
- link panda_rightfinger: geometry collision mesh filename=package://robots/franka_panda/meshes/collision/finger.stl; visual mesh filename=package://robots/franka_panda/meshes/visual/finger.dae
- link shoulder_link: geometry collision mesh filename=package://robots/ur5/meshes/collision/shoulder.stl; visual mesh filename=package://robots/ur5/meshes/visual/shoulder.dae
- link upper_arm_link: geometry collision mesh filename=package://robots/ur5/meshes/collision/upperarm.stl; visual mesh filename=package://robots/ur5/meshes/visual/upperarm.dae
- link wrist_1_link: geometry collision mesh filename=package://robots/ur5/meshes/collision/wrist1.stl; visual mesh filename=package://robots/ur5/meshes/visual/wrist1.dae
- link wrist_2_link: geometry collision mesh filename=package://robots/ur5/meshes/collision/wrist2.stl; visual mesh filename=package://robots/ur5/meshes/visual/wrist2.dae
- link wrist_3_link: geometry collision mesh filename=package://robots/ur5/meshes/collision/wrist3.stl; visual mesh filename=package://robots/ur5/meshes/visual/wrist3.dae
