Commit message: adding static fingers to panda robot

File: src/guided_tamp_benchmark/models/data/robots/franka_panda/panda_pddl.urdf (robot description, URDF)
Before this commit: robot panda, 10 links, 9 joints
Links:
- added link panda_leftfinger, mass 0.1; collision mesh filename=package://robots/franka_panda/meshes/collision/finger.stl; visual mesh filename=package://robots/franka_panda/meshes/visual/finger.dae
- added link panda_rightfinger, mass 0.1; collision mesh filename=package://robots/franka_panda/meshes/collision/finger.stl; visual mesh filename=package://robots/franka_panda/meshes/visual/finger.dae
Joints:
- added joint panda_finger_joint1: type fixed, parent panda_hand, child panda_leftfinger, origin xyz=0 0.04 0.0584 rpy=0 0 0
- added joint panda_finger_joint2: type fixed, parent panda_hand, child panda_rightfinger, origin xyz=0 -0.04 0.0584 rpy=0 0 0, mimic joint=panda_finger_joint1
