Commit message: Changes to mobile robot

File: src/guided_tamp_benchmark/models/data/robots/kuka_kmr_iiwa/kuka_kmr_iiwa.urdf (robot description, URDF)
Before this commit: robot kmr_iiwa, 16 links, 15 joints
Joints:
- joint help_0_to_help_1: limit lower=-5 upper=5 effort=100 velocity=1 -> lower=-0.5 upper=4 effort=100 velocity=1
- joint world_to_help_0: limit lower=-5 upper=5 effort=100 velocity=1 -> lower=-2 upper=3 effort=100 velocity=1

Commit message: Modify mobile robot configuration

File: src/guided_tamp_benchmark/models/data/robots/kuka_kmr_iiwa/kuka_kmr_iiwa.urdf (robot description, URDF)
Before this commit: robot kmr_iiwa, 16 links, 15 joints
Joints:
- joint help_0_to_help_1: limit lower=-0.5 upper=4 effort=100 velocity=1 -> lower=0.75 upper=2.45 effort=100 velocity=1
- joint world_to_help_0: limit lower=-2 upper=3 effort=100 velocity=1 -> lower=-0.5 upper=1.25 effort=100 velocity=1

Commit message: increase limits for kmr robot

File: src/guided_tamp_benchmark/models/data/robots/kuka_kmr_iiwa/kuka_kmr_iiwa.urdf (robot description, URDF)
Before this commit: robot kmr_iiwa, 16 links, 15 joints
Joints:
- removed joint help_0_to_help_1
- removed joint help_1_to_kmr
- removed joint world_to_help_0
- added joint help_0_to_help_1_joint: type prismatic, parent help_link_0, child help_link_1, origin xyz=0 0 0 rpy=0 0 0, axis 0 1 0, limit lower=-3 upper=3 effort=100 velocity=1
- added joint help_1_to_kmr_joint: type revolute, parent help_link_1, child kmr_link, origin xyz=0 0 0 rpy=0 0 0, axis 0 0 1, limit lower=-5 upper=5 effort=100 velocity=1
- added joint world_to_help_0_joint: type prismatic, parent world, child help_link_0, origin xyz=0 0 0 rpy=0 0 0, axis 1 0 0, limit lower=-3 upper=3 effort=100 velocity=1
