Commit message: Swith PandaRobot to camera panda version and change gripper orientation at grasp

File: guided_tamp_benchmark/models/data/robots/franka_panda/panda_camera.urdf (robot description, URDF)
Before this commit: robot panda, 12 links, 11 joints
Links:
- added link panda_camera_mount, mass 0.1; collision box size=0.05 0.13 0.07; visual box size=0.03 0.10 0.04
Joints:
- added joint panda_camera_mount_joint: type fixed, parent panda_link8, child panda_camera_mount, origin xyz=0 0 0 rpy=0 0 -0.7853981633974483
- joint panda_finger_joint1: limit lower=0.0 upper=0.04 effort=20 velocity=0.2 -> lower=0.0 upper=0.041 effort=20 velocity=0.2
- joint panda_finger_joint2: limit lower=0.0 upper=0.04 effort=20 velocity=0.2 -> lower=0.0 upper=0.041 effort=20 velocity=0.2
- joint panda_joint2: limit lower=-1.8326 upper=1.8326 effort=87 velocity=2.1750 -> lower=-1.6628 upper=1.6628 effort=87 velocity=2.3925
- joint panda_joint3: limit lower=-2.9671 upper=2.9671 effort=87 velocity=2.1750 -> lower=-2.7973 upper=2.7973 effort=87 velocity=2.3925
- joint panda_joint4: limit lower=-3.1416 upper=0.0 effort=87 velocity=2.1750 -> lower=-2.9718 upper=-0.0825 effort=87 velocity=2.3925
- joint panda_joint5: limit lower=-2.9671 upper=2.9671 effort=12 velocity=2.6100 -> lower=-2.7973 upper=2.7973 effort=12 velocity=2.8710
- joint panda_joint6: limit lower=-0.0873 upper=3.8223 effort=12 velocity=2.6100 -> lower=0.0825 upper=3.6525 effort=12 velocity=2.8710
- joint panda_joint7: limit lower=-2.9671 upper=2.9671 effort=12 velocity=2.6100 -> lower=-2.7973 upper=2.7973 effort=12 velocity=2.8710
